File: PCB/magnetics.kicad_sch (KiCad schematic)
At the start: 0 parts

Commit message: realized the magnetic sensor wont work because of orientation
Parts:
- added C1: ~, symbol Device:C
- added MAG1: TMAG6180EDGKRQ1, TMAG6180:VSSOP8_3P1X3P1_TEX, symbol TMAG6180:TMAG6180EDGKRQ1
- added R1, R2, R3, R4: R_Small_US, Resistor_SMD:R_0402_1005Metric, symbol Device:R_Small_US
Connections:
- new net +3.3V: C1.1, MAG1.7 (VCC)
- new net COS_N: MAG1.3 (COS_N), R1.2
- new net COS_P: MAG1.1 (COS_P), R2.2
- new net GND: C1.2, MAG1.2 (GND), R1.1, R2.1, R3.1, R4.1
- new net SIN_N: MAG1.6 (SIN_N), R4.2
- new net SIN_P: MAG1.8 (SIN_P), R3.2
- no-connect marks 0 -> 2
Other:
- note added: "angle = arctan^(2)(Vsin/Vcos)/2"
